Commit message: Fixed collision model of kinect sensor urdf

File: uibk_robot/urdf/sensor_kinect.xacro (robot description, xacro)
@@ -53,5 +53,6 @@
       </visual>
       <collision>
-	<origin xyz="-0.0315 0.0 -0.017" rpy="0 0 0"/>
+	<!--origin xyz="-0.0315 0.0 -0.017" rpy="0 0 0"/-->
+	<origin xyz="0 0 0.0365" rpy="0 0 ${M_PI/2}"/>
 	<geometry>
 	  <box size="0.07271 0.27794 0.073"/>

File: uibk_robot/urdf/torso.xacro (robot description, xacro)
@@ -17,5 +17,5 @@
       <collision>
 	<geometry>
-	  <mesh filename="package://uibk_robot/meshes/torso_convex.stl"/>
+	  <mesh filename="package://uibk_robot/meshes/torso_convex2.stl"/>
 	</geometry>
       </collision>

Commit message: Fixed collision model in sensor_kinect

File: uibk_robot/urdf/sensor_kinect.xacro (robot description, xacro)
@@ -53,5 +53,5 @@
       </visual>
       <collision>
-	<origin xyz="-0.0315 0.0 -0.017" rpy="0 0 0"/>
+	<origin xyz="0 0 0.0365" rpy="0 0 ${M_PI/2}"/>
 	<geometry>
 	  <box size="0.07271 0.27794 0.073"/>
