Commit message: Included KIT head into urdf model

File: uibk_robot/urdf/uibk_robot.xacro (robot description, xacro)
@@ -1,9 +1,9 @@
 <?xml version="1.0"?>
 <robot xmlns:xacro="http://www.ros.org/wiki/xacro" name="uibk_robot">
-  <xacro:include filename="materials.urdf"/>
   <xacro:include filename="torso.xacro"/>
   <xacro:include filename="table.xacro"/>
-  <xacro:include filename="kuka_lwr_arm_defs.xacro"/>
   <xacro:include filename="sdh_with_connector.xacro"/>
+  <xacro:include filename="$(find lwr_description)/urdf/kuka_lwr_arm_defs.xacro"/>
+  <xacro:include filename="$(find kit_head_description)/model/kit_head.urdf.xacro" />
   <!-- draw a small cross to visualize the origin of the world reference frame -->
   <link name="world_link">
@@ -41,3 +41,7 @@
     <origin rpy="0 0 ${1/2 * M_PI}"/>
   </xacro:sdh_with_connector>
+  <!-- HEAD -->
+  <xacro:kit_head name="head" parent="world">
+    <origin xyz="-0.4723 0.6767 0.85"/>
+  </xacro:kit_head>
 </robot>

File: uibk_robot/urdf/uibk_robot_left_sdh.xacro (robot description, xacro)
@@ -1,10 +1,10 @@
 <?xml version="1.0"?>
 <robot xmlns:xacro="http://www.ros.org/wiki/xacro" name="uibk_robot">
-  <xacro:include filename="materials.urdf"/>
   <xacro:include filename="torso.xacro"/>
   <xacro:include filename="table.xacro"/>
-  <xacro:include filename="kuka_lwr_arm_defs.xacro"/>
   <xacro:include filename="sdh_with_connector.xacro"/>
   <xacro:include filename="dummy_eef.xacro"/>
+  <xacro:include filename="$(find lwr_description)/urdf/kuka_lwr_arm_defs.xacro"/>
+  <xacro:include filename="$(find kit_head_description)/model/kit_head.urdf.xacro" />
   <!-- draw a small cross to visualize the origin of the world reference frame -->
   <link name="world_link">
@@ -51,3 +51,7 @@
     <origin rpy="0 0 0"/>
   </xacro:dummy_eef>
+  <!-- HEAD -->
+  <xacro:kit_head name="head" parent="world">
+    <origin xyz="-0.4723 0.6767 0.85"/>
+  </xacro:kit_head>
 </robot>

File: uibk_robot/urdf/uibk_robot_right_sdh.xacro (robot description, xacro)
@@ -1,10 +1,10 @@
 <?xml version="1.0"?>
 <robot xmlns:xacro="http://www.ros.org/wiki/xacro" name="uibk_robot">
-  <xacro:include filename="materials.urdf"/>
   <xacro:include filename="torso.xacro"/>
   <xacro:include filename="table.xacro"/>
-  <xacro:include filename="kuka_lwr_arm_defs.xacro"/>
   <xacro:include filename="sdh_with_connector.xacro"/>
   <xacro:include filename="dummy_eef.xacro"/>
+  <xacro:include filename="$(find lwr_description)/urdf/kuka_lwr_arm_defs.xacro"/>
+  <xacro:include filename="$(find kit_head_description)/model/kit_head.urdf.xacro" />
   <!-- draw a small cross to visualize the origin of the world reference frame -->
   <link name="world_link">
@@ -51,3 +51,7 @@
     <origin rpy="0 0 ${1/2 * M_PI}"/>
   </xacro:sdh_with_connector>
+  <!-- HEAD -->
+  <xacro:kit_head name="head" parent="world">
+    <origin xyz="-0.4723 0.6767 0.85"/>
+  </xacro:kit_head>
 </robot>

File: uibk_robot/urdf/uibk_robot_table.xacro (robot description, xacro)
@@ -1,9 +1,9 @@
 <?xml version="1.0"?>
 <robot xmlns:xacro="http://www.ros.org/wiki/xacro" name="uibk_robot">
-  <xacro:include filename="materials.urdf"/>
   <xacro:include filename="torso.xacro"/>
   <xacro:include filename="table.xacro"/>
-  <xacro:include filename="kuka_lwr_arm_defs.xacro"/>
   <xacro:include filename="sdh_with_connector.xacro"/>
+  <xacro:include filename="$(find lwr_description)/urdf/kuka_lwr_arm_defs.xacro"/>
+  <xacro:include filename="$(find kit_head_description)/model/kit_head.urdf.xacro" />
   <!-- draw a small cross to visualize the origin of the world reference frame -->
   <link name="world_link">
@@ -50,4 +50,8 @@
     <origin rpy="0 0 ${1/2 * M_PI}"/>
   </xacro:sdh_with_connector>
+  <!-- HEAD -->
+  <xacro:kit_head name="head" parent="world">
+    <origin xyz="-0.4723 0.6767 0.85"/>
+  </xacro:kit_head>
   <!-- Kinect vision sensor -->
   <!-- <link name="camera_link"/>
